File: hardware/E200.sch (EAGLE design)
At the start: 26 parts, among them SW1 SPST_TACT-KMR2, U11 915MHz, U5 ATMEGA328P-MU, U8 MCP1703CB, X1 16 MHz

Commit message: v1.1.0 - small update
- added silkscreen to bottom for node id
- solder mask DRU for covering vias
- removed solder jumper
- minor trace adjustments
- functionally same as previous
Parts:
- removed SS: JUMPER-SMT_2_NC_PASTE_SILK, SparkFun-Jumpers:JUMPER-SMT_2_NC_PASTE_SILK
Connections:
- removed net N$11: R7.2, SS.2
- net VCC: now also R7.2; no longer SS.1
Changed lines of the file:
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@@
 <?xml version="1.0" encoding="utf-8"?>
 <!DOCTYPE eagle SYSTEM "eagle.dtd">
-<eagle version="9.4.1">
+<eagle version="9.5.1">
 <drawing>
 <settings>
@@
 <part name="SUPPLY9" library="SparkFun-Aesthetics" deviceset="VCC" device=""/>
 <part name="GND6" library="SparkFun-Aesthetics" deviceset="GND" device=""/>
-<part name="SS" library="SparkFun-Jumpers" deviceset="JUMPER-SMT_2_NC_PASTE" device="_SILK"/>
 <part name="D1" library="SCHOTTKY_0805" deviceset="DIODE_SCHOTTKY" device="0805-RES"/>
 </parts>
@@
 <attribute name="VALUE" x="132.08" y="99.06" size="1.778" layer="96"/>
 </instance>
-<instance part="SS" gate="G$1" x="210.82" y="43.18" smashed="yes" rot="R270">
-<attribute name="NAME" x="213.36" y="45.72" size="1.778" layer="95" font="vector" rot="R270"/>
-<attribute name="VALUE" x="208.28" y="45.72" size="1.778" layer="96" font="vector" rot="R270" align="top-left"/>
-</instance>
 <instance part="D1" gate="G$1" x="241.3" y="-43.18" smashed="yes">
 <attribute name="NAME" x="237.49" y="-41.4274" size="1.778" layer="95"/>
@@
 </segment>
 <segment>
-<wire x1="210.82" y1="48.26" x2="210.82" y2="50.8" width="0.1524" layer="91"/>
-<pinref part="SUPPLY2" gate="G$1" pin="VCC"/>
-<pinref part="SS" gate="G$1" pin="1"/>
-</segment>
-<segment>
 <pinref part="JP2" gate="A" pin="2"/>
 <wire x1="149.86" y1="109.22" x2="134.62" y2="109.22" width="0.1524" layer="91"/>
 <wire x1="134.62" y1="109.22" x2="134.62" y2="119.38" width="0.1524" layer="91"/>
 <pinref part="SUPPLY9" gate="G$1" pin="VCC"/>
+</segment>
+<segment>
+<pinref part="R7" gate="G$1" pin="2"/>
+<pinref part="SUPPLY2" gate="G$1" pin="VCC"/>
+<wire x1="210.82" y1="35.56" x2="210.82" y2="50.8" width="0.1524" layer="91"/>
 </segment>
 </net>
@@
 </segment>
 </net>
-<net name="N$11" class="0">
-<segment>
-<pinref part="R7" gate="G$1" pin="2"/>
-<wire x1="210.82" y1="35.56" x2="210.82" y2="38.1" width="0.1524" layer="91"/>
-<pinref part="SS" gate="G$1" pin="2"/>
-</segment>
-</net>
